File: ZT1 Schematics/Oscillator.kicad_sch (KiCad schematic)
At the start: 14 parts, among them U132 74LS10, U136 74LS04, U142 74LS161, X101 Crystal

Commit message: Minor touchups
Fixed some of the text
Added some explanations
Simplified the video circuit
Parts:
- C108, C109, C110: footprint ZX1:C_Disc_D9.0mm_W2.5mm_P7.50mm -> ZT1:C_Disc_D9.0mm_W2.5mm_P7.50mm
- C111, C119, C121, C152: footprint ZX1:C_350mil -> ZT1:C_350mil
- L104: footprint ZX1:L_Axial_L7.0mm_D3.3mm_P5.08mm_Vertical_Fastron_MICC -> ZT1:L_Axial_L7.0mm_D3.3mm_P5.08mm_Vertical_Fastron_MICC
- R128, R129: footprint ZX1:R_450mil -> ZT1:R_450mil
Changed lines of the file:
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@@
 			)
 		)
-		(property "Footprint" "ZX1:R_450mil"
+		(property "Footprint" "ZT1:R_450mil"
 			(at 88.9 80.518 90)
 			(effects
@@
 			)
 		)
-		(property "Datasheet" ""
+		(property "Datasheet" "~"
 			(at 88.9 78.74 0)
 			(effects
@@
 			)
 		)
-		(property "Description" ""
+		(property "Description" "Resistor"
 			(at 88.9 78.74 0)
 			(effects
@@
 		)
 		(instances
-			(project "ZX1"
+			(project "ZT1"
 				(path "/f4096561-d684-4672-ab54-4b1ef20fc4c8/1522dedb-184f-4914-b2e2-907c84c4788d"
 					(reference "R129")
@@
 			)
 		)
-		(property "Footprint" "ZX1:C_Disc_D9.0mm_W2.5mm_P7.50mm"
+		(property "Footprint" "ZT1:C_Disc_D9.0mm_W2.5mm_P7.50mm"
 			(at 83.5152 88.9 0)
 			(effects
@@
 			)
 		)
-		(property "Datasheet" ""
+		(property "Datasheet" "~"
 			(at 82.55 85.09 0)
 			(effects
@@
 			)
 		)
-		(property "Description" ""
+		(property "Description" "Unpolarized capacitor"
 			(at 82.55 85.09 0)
 			(effects
@@
 		)
 		(instances
-			(project "ZX1"
+			(project "ZT1"
 				(path "/f4096561-d684-4672-ab54-4b1ef20fc4c8/1522dedb-184f-4914-b2e2-907c84c4788d"
 					(reference "C109")
@@
 		)
 		(instances
-			(project "ZX1"
+			(project "ZT1"
 				(path "/f4096561-d684-4672-ab54-4b1ef20fc4c8/1522dedb-184f-4914-b2e2-907c84c4788d"
 					(reference "U142")
@@
 			)
 		)
-		(property "Footprint" "ZX1:C_350mil"
+		(property "Footprint" "ZT1:C_350mil"
 			(at 97.4852 30.48 0)
 			(effects
@@
 			)
 		)
-		(property "Datasheet" ""
+		(property "Datasheet" "~"
 			(at 96.52 26.67 0)
 			(effects
@@
 			)
 		)
-		(property "Description" ""
+		(property "Description" "Unpolarized capacitor"
 			(at 96.52 26.67 0)
 			(effects
@@
 			)
 		)
-		(property "Footprint" "ZX1:R_450mil"
+		(property "Footprint" "ZT1:R_450mil"
 			(at 76.2 80.518 90)
 			(effects
@@
 			)
 		)
-		(property "Datasheet" ""
+		(property "Datasheet" "~"
 			(at 76.2 78.74 0)
 			(effects
@@
 			)
 		)
-		(property "Description" ""
+		(property "Description" "Resistor"
 			(at 76.2 78.74 0)
 			(effects
@@
 		)
 		(instances
-			(project "ZX1"
+			(project "ZT1"
 				(path "/f4096561-d684-4672-ab54-4b1ef20fc4c8/1522dedb-184f-4914-b2e2-907c84c4788d"
 					(reference "#PWR023")
@@
 	)
 	(symbol
-		(lib_name "74LS10_1")
 		(lib_id "74xx:74LS10")
 		(at 162.56 35.56 270)
@@
 		)
 		(instances
-			(project "ZX1"
+			(project "ZT1"
 				(path "/f4096561-d684-4672-ab54-4b1ef20fc4c8/1522dedb-184f-4914-b2e2-907c84c4788d"
 					(reference "U132")
@@
 			)
 		)
-		(property "Footprint" "ZX1:C_350mil"
+		(property "Footprint" "ZT1:C_350mil"
 			(at 78.4352 30.48 0)
 			(effects
@@
 			)
 		)
-		(property "Datasheet" ""
+		(property "Datasheet" "~"
 			(at 77.47 26.67 0)
 			(effects
@@
 			)
 		)
-		(property "Description" ""
+		(property "Description" "Unpolarized capacitor"
 			(at 77.47 26.67 0)
 			(effects
@@
 		)
 		(instances
-			(project "ZX1"
+			(project "ZT1"
 				(path "/f4096561-d684-4672-ab54-4b1ef20fc4c8/1522dedb-184f-4914-b2e2-907c84c4788d"
 					(reference "#PWR08")
@@
 		)
 		(instances
-			(project "ZX1"
+			(project "ZT1"
 				(path "/f4096561-d684-4672-ab54-4b1ef20fc4c8/1522dedb-184f-4914-b2e2-907c84c4788d"
 					(reference "#PWR013")
@@
 		)
 		(instances
-			(project "ZX1"
+			(project "ZT1"
 				(path "/f4096561-d684-4672-ab54-4b1ef20fc4c8/1522dedb-184f-4914-b2e2-907c84c4788d"
 					(reference "#PWR07")
@@
 			)
 		)
-		(property "Datasheet" ""
+		(property "Datasheet" "~"
 			(at 82.55 52.07 0)
 			(effects
@@
 			)
 		)
-		(property "Description" ""
+		(property "Description" "Two pin crystal"
 			(at 82.55 52.07 0)
 			(effects
@@
 			)
 		)
-		(property "Footprint" "ZX1:C_Disc_D9.0mm_W2.5mm_P7.50mm"
+		(property "Footprint" "ZT1:C_Disc_D9.0mm_W2.5mm_P7.50mm"
 			(at 70.8152 88.9 0)
 			(effects
@@
 			)
 		)
-		(property "Datasheet" ""
+		(property "Datasheet" "~"
 			(at 69.85 85.09 0)
 			(effects
@@
 			)
 		)
-		(property "Description" ""
+		(property "Description" "Unpolarized capacitor"
 			(at 69.85 85.09 0)
 			(effects
@@
 		)
 		(instances
-			(project "ZX1"
+			(project "ZT1"
 				(path "/f4096561-d684-4672-ab54-4b1ef20fc4c8/1522dedb-184f-4914-b2e2-907c84c4788d"
 					(reference "U132")
@@
 			)
 		)
-		(property "Footprint" "ZX1:C_350mil"
+		(property "Footprint" "ZT1:C_350mil"
 			(at 152.4 33.3248 0)
 			(effects
@@
 			)
 		)
-		(property "Datasheet" ""
+		(property "Datasheet" "~"
 			(at 148.59 34.29 0)
 			(effects
@@
 			)
 		)
-		(property "Description" ""
+		(property "Description" "Unpolarized capacitor"
 			(at 148.59 34.29 0)
 			(effects
@@
 			)
 		)
-		(property "Footprint" "ZX1:C_Disc_D9.0mm_W2.5mm_P7.50mm"
+		(property "Footprint" "ZT1:C_Disc_D9.0mm_W2.5mm_P7.50mm"
 			(at 96.2152 88.9 0)
 			(effects
@@
 			)
 		)
-		(property "Datasheet" ""
+		(property "Datasheet" "~"
 			(at 95.25 85.09 0)
 			(effects
@@
 			)
 		)
-		(property "Description" ""
+		(property "Description" "Unpolarized capacitor"
 			(at 95.25 85.09 0)
 			(effects
@@
 		)
 		(instances
-			(project "ZX1"
+			(project "ZT1"
 				(path "/f4096561-d684-4672-ab54-4b1ef20fc4c8/1522dedb-184f-4914-b2e2-907c84c4788d"
 					(reference "C110")
@@
 			)
 		)
-		(property "Footprint" "ZX1:L_Axial_L7.0mm_D3.3mm_P5.08mm_Vertical_Fastron_MICC"
+		(property "Footprint" "ZT1:L_Axial_L7.0mm_D3.3mm_P5.08mm_Vertical_Fastron_MICC"
 			(at 87.63 21.59 0)
 			(effects
@@
 			)
 		)
-		(property "Datasheet" ""
+		(property "Datasheet" "~"
 			(at 87.63 21.59 0)
 			(effects
@@
 			)
 		)
-		(property "Description" ""
+		(property "Description" "Inductor"
 			(at 87.63 21.59 0)
 			(effects
@@
 			)
 		)
-		(property "Footprint" "ZX1:C_350mil"
+		(property "Footprint" "ZT1:C_350mil"
 			(at 23.8252 31.75 0)
 			(effects
@@
 			)
 		)
-		(property "Datasheet" ""
+		(property "Datasheet" "~"
 			(at 22.86 27.94 0)
 			(effects
@@
 			)
 		)
-		(property "Description" ""
+		(property "Description" "Unpolarized capacitor"
 			(at 22.86 27.94 0)
 			(effects
