File: ZT1 Schematics/VRAM.kicad_sch (KiCad schematic)
At the start: 13 parts, among them U103 74LS02, U106 74LS32, U107 74LS08, U108 74LS00, U119 74LS245, U124 D2114LC, U125 D2114LC, U126 HM6116P, U127 7432

Commit message: Minor touchups
Fixed some of the text
Added some explanations
Simplified the video circuit
Parts:
- C134, C135, C136, C137: footprint ZX1:C_350mil -> ZT1:C_350mil
- U124, U125: symbol ZX1:D2114LC -> ZT1:D2114LC
- U126: symbol ZX1:HM6116P -> ZT1:HM6116P
Changed lines of the file:
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@@
 			)
 		)
-		(property "Footprint" "ZX1:C_350mil"
+		(property "Footprint" "ZT1:C_350mil"
 			(at 217.17 108.2548 0)
 			(effects
@@
 			)
 		)
-		(property "Datasheet" ""
+		(property "Datasheet" "~"
 			(at 213.36 109.22 0)
 			(effects
@@
 			)
 		)
-		(property "Description" ""
+		(property "Description" "Unpolarized capacitor"
 			(at 213.36 109.22 0)
 			(effects
@@
 	)
 	(symbol
-		(lib_id "ZX1:HM6116P")
+		(lib_id "ZT1:HM6116P")
 		(at 162.56 114.3 0)
 		(unit 1)
@@
 			)
 		)
-		(property "Footprint" "ZX1:C_350mil"
+		(property "Footprint" "ZT1:C_350mil"
 			(at 251.1552 104.14 0)
 			(effects
@@
 			)
 		)
-		(property "Datasheet" ""
+		(property "Datasheet" "~"
 			(at 250.19 100.33 0)
 			(effects
@@
 			)
 		)
-		(property "Description" ""
+		(property "Description" "Unpolarized capacitor"
 			(at 250.19 100.33 0)
 			(effects
@@
 			)
 		)
-		(property "Footprint" "ZX1:C_350mil"
+		(property "Footprint" "ZT1:C_350mil"
 			(at 218.1352 68.58 0)
 			(effects
@@
 			)
 		)
-		(property "Datasheet" ""
+		(property "Datasheet" "~"
 			(at 217.17 64.77 0)
 			(effects
@@
 			)
 		)
-		(property "Description" ""
+		(property "Description" "Unpolarized capacitor"
 			(at 217.17 64.77 0)
 			(effects
@@
 	)
 	(symbol
-		(lib_id "ZX1:D2114LC")
+		(lib_id "ZT1:D2114LC")
 		(at 204.47 80.01 0)
 		(unit 1)
@@
 		)
 		(instances
-			(project "ZX1"
+			(project "ZT1"
 				(path "/f4096561-d684-4672-ab54-4b1ef20fc4c8/1b0cf4c1-249a-46f4-a9d3-5c0e911316e3"
 					(reference "U127")
@@
 			)
 		)
-		(property "Footprint" "ZX1:C_350mil"
+		(property "Footprint" "ZT1:C_350mil"
 			(at 177.8 84.1248 0)
 			(effects
@@
 			)
 		)
-		(property "Datasheet" ""
+		(property "Datasheet" "~"
 			(at 173.99 85.09 0)
 			(effects
@@
 			)
 		)
-		(property "Description" ""
+		(property "Description" "Unpolarized capacitor"
 			(at 173.99 85.09 0)
 			(effects
@@
 		)
 		(instances
-			(project "ZX1"
+			(project "ZT1"
 				(path "/f4096561-d684-4672-ab54-4b1ef20fc4c8/1b0cf4c1-249a-46f4-a9d3-5c0e911316e3"
 					(reference "U127")
@@
 		)
 		(instances
-			(project "ZX1"
+			(project "ZT1"
 				(path "/f4096561-d684-4672-ab54-4b1ef20fc4c8/1b0cf4c1-249a-46f4-a9d3-5c0e911316e3"
 					(reference "U108")
@@
 	)
 	(symbol
-		(lib_id "ZX1:D2114LC")
+		(lib_id "ZT1:D2114LC")
 		(at 204.47 132.08 0)
 		(unit 1)
@@
 		)
 		(instances
-			(project "ZX1"
+			(project "ZT1"
 				(path "/f4096561-d684-4672-ab54-4b1ef20fc4c8/1b0cf4c1-249a-46f4-a9d3-5c0e911316e3"
 					(reference "U103")
